File: cad/push-on-hold-off.kicad_pcb (KiCad board)
At the start: 2 copper layers, 22.9 x 12.7 mm, 11 parts, among them P1 CONN_01X04, P2 CONN_01X04, Q1 IRF7309IPBF, SW1 SW_PUSH_SMALL

Commit message: Add silkscreen connection reference
Other:
- board text added: "BUT"
- board text added: "GND"
- board text added: "Vin"
- board text added: "Vout"
Changed lines of the file:
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@@
     (links 27)
     (no_connects 0)
-    (area 213.331667 98.645 241.328334 114.565)
+    (area 215.824999 100.254999 238.835001 113.105001)
     (thickness 1.6)
-    (drawings 8)
+    (drawings 16)
     (tracks 128)
     (zones 0)
@@
   (page A4)
   (layers
-    (0 F.Cu signal)
+    (0 F.Cu signal hide)
     (31 B.Cu signal)
     (32 B.Adhes user)
@@
     (aux_axis_origin 0 0)
     (grid_origin 217.175 100.345)
-    (visible_elements 7FFFFFFF)
+    (visible_elements 7FFFBFFF)
     (pcbplotparams
-      (layerselection 0x000f0_80000001)
+      (layerselection 0x010f0_80000001)
       (usegerberextensions true)
       (excludeedgelayer true)
@@
     )
   )
+  (gr_text Vout (at 233.177 110.505) (layer B.SilkS)
+    (effects (font (size 1 1) (thickness 0.25)) (justify mirror))
+  )
+  (gr_text BUT (at 233.685 107.965) (layer B.SilkS)
+    (effects (font (size 1 1) (thickness 0.25)) (justify mirror))
+  )
+  (gr_text GND (at 233.685 105.425) (layer B.SilkS)
+    (effects (font (size 1 1) (thickness 0.25)) (justify mirror))
+  )
+  (gr_text GND (at 233.431 102.885) (layer B.SilkS)
+    (effects (font (size 1 1) (thickness 0.25)) (justify mirror))
+  )
+  (gr_text Vin (at 221.239 110.505) (layer B.SilkS)
+    (effects (font (size 1 1) (thickness 0.25)) (justify mirror))
+  )
+  (gr_text BUT (at 221.239 107.965) (layer B.SilkS)
+    (effects (font (size 1 1) (thickness 0.25)) (justify mirror))
+  )
+  (gr_text GND (at 221.239 105.425) (layer B.SilkS)
+    (effects (font (size 1 1) (thickness 0.25)) (justify mirror))
+  )
+  (gr_text GND (at 221.239 102.885) (layer B.SilkS)
+    (effects (font (size 1 1) (thickness 0.25)) (justify mirror))
+  )
   (gr_line (start 237.49 100.33) (end 217.17 100.33) (angle 90) (layer Edge.Cuts) (width 0.15))
